Commit message: xacro variable introduction

File: src/my_robot_description/urdf/my_robot.urdf.xacro (robot description, xacro)
@@ -1,4 +1,5 @@
 <?xml version="1.0"?>
 <robot name="my_robot" xmlns:xacro="https://www.ros.org/wiki/xacro">
+    <xacro:property name="base_length" value="0.6"/>
     <material name="blue">
         <color rgba="0 0 0.5 1"/>
@@ -10,5 +11,5 @@
         <visual>
             <geometry>
-                <box size="0.6 0.4 0.2" />
+                <box size="${base_length} 0.4 0.2" />
             </geometry>
             <origin xyz="0 0 0.1" rpy="0 0 0" />
@@ -19,5 +20,5 @@
         <parent link="base_link"/>
         <child link = "right_wheel_link"/>
-        <origin xyz="-0.15 -0.225 0" rpy="0 0 0"/>
+        <origin xyz="${-base_length/4} -0.225 0" rpy="0 0 0"/>
         <axis xyz="0 1 0"/>
     </joint>
@@ -27,5 +28,5 @@
                 <cylinder radius="0.1" length="0.05"/>
             </geometry>
-            <origin xyz="0 0 0" rpy="1.57 0 0"/>
+            <origin xyz="0 0 0" rpy="${pi/2.0} 0 0"/>
             <material name="grey"/>
         </visual>
@@ -34,5 +35,5 @@
         <parent link="base_link"/>
         <child link = "left_wheel_link"/>
-        <origin xyz="-0.15 0.225 0" rpy="0 0 0"/>
+        <origin xyz="${-base_length/4} 0.225 0" rpy="0 0 0"/>
         <axis xyz="0 1 0"/>
     </joint>
@@ -42,5 +43,5 @@
                 <cylinder radius="0.1" length="0.05"/>
             </geometry>
-            <origin xyz="0 0 0" rpy="1.57 0 0"/>
+            <origin xyz="0 0 0" rpy="${pi/2.0} 0 0"/>
             <material name="grey"/>
         </visual>
@@ -49,5 +50,5 @@
         <parent link="base_link"/>
         <child link = "caster_wheel_link"/>
-        <origin xyz="0.2 0 -0.05" rpy="0 0 0"/>
+        <origin xyz="${base_length/3} 0 -0.05" rpy="0 0 0"/>
     </joint>
     <link name="caster_wheel_link">

Commit message: Xacro functions, and nested xacro files

File: src/my_robot_description/urdf/my_robot.urdf.xacro (robot description, xacro)
@@ -1,73 +1,5 @@
 <?xml version="1.0"?>
 <robot name="my_robot" xmlns:xacro="https://www.ros.org/wiki/xacro">
-    <xacro:property name="base_length" value="0.6"/>
-    <material name="blue">
-        <color rgba="0 0 0.5 1"/>
-    </material>
-    <material name="grey">
-        <color rgba="0.5 0.5 0.5 1"/>
-    </material>
-    <link name="base_link">
-        <visual>
-            <geometry>
-                <box size="${base_length} 0.4 0.2" />
-            </geometry>
-            <origin xyz="0 0 0.1" rpy="0 0 0" />
-            <material name="blue" />
-        </visual>
-    </link>
-    <joint name = "base_right_wheel_joint" type="continuous">
-        <parent link="base_link"/>
-        <child link = "right_wheel_link"/>
-        <origin xyz="${-base_length/4} -0.225 0" rpy="0 0 0"/>
-        <axis xyz="0 1 0"/>
-    </joint>
-    <link name="right_wheel_link">
-        <visual>
-            <geometry>
-                <cylinder radius="0.1" length="0.05"/>
-            </geometry>
-            <origin xyz="0 0 0" rpy="${pi/2.0} 0 0"/>
-            <material name="grey"/>
-        </visual>
-    </link>
-    <joint name = "base_left_wheel_joint" type="continuous">
-        <parent link="base_link"/>
-        <child link = "left_wheel_link"/>
-        <origin xyz="${-base_length/4} 0.225 0" rpy="0 0 0"/>
-        <axis xyz="0 1 0"/>
-    </joint>
-    <link name="left_wheel_link">
-        <visual>
-            <geometry>
-                <cylinder radius="0.1" length="0.05"/>
-            </geometry>
-            <origin xyz="0 0 0" rpy="${pi/2.0} 0 0"/>
-            <material name="grey"/>
-        </visual>
-    </link>
-    <joint name = "base_caster_wheel_joint" type="fixed">
-        <parent link="base_link"/>
-        <child link = "caster_wheel_link"/>
-        <origin xyz="${base_length/3} 0 -0.05" rpy="0 0 0"/>
-    </joint>
-    <link name="caster_wheel_link">
-        <visual>
-            <geometry>
-                <sphere radius="0.05"/>
-            </geometry>
-            <origin xyz="0 0 0" rpy="0 0 0"/>
-            <material name="grey"/>
-        </visual>
-    </link>
-    <joint name = "base_joint" type="fixed">
-        <parent link="base_footprint"/>
-        <child link = "base_link"/>
-        <origin xyz="0 0 0.1" rpy="0 0 0"/>
-    </joint>
-    <link name="base_footprint">
-        <visual>
-            <origin xyz="0 0 0" rpy="0 0 0"/>
-        </visual>
-    </link>
+    <xacro:include filename="common_properties.xacro"/>
+    <xacro:include filename="mobile_base.xacro"/>
 </robot>
