Commit message: gazebo_ros package

File: src/my_robot_description/urdf/mobile_base.xacro (robot description, xacro)
@@ -14,4 +14,10 @@
             <material name="blue" />
         </visual>
+        <collision>
+            <geometry>
+                <box size="${base_length} ${base_width} ${base_height}" />
+            </geometry>
+            <origin xyz="0 0 ${base_height / 2.0}" rpy="0 0 0" />
+        </collision>
         <xacro:box_inertia  m="5" l="${base_length}" w="${base_width}" h="${base_height}"
                             xyz="0 0 ${base_height/2.0}" rpy="0 0 0"/>
@@ -32,4 +38,10 @@
                 <material name="grey"/>
             </visual>
+            <collision>
+                <geometry>
+                    <cylinder radius="${wheel_radius}" length="${wheel_length}"/>
+                </geometry>
+                <origin xyz="0 0 0" rpy="${pi/2.0} 0 0"/>
+            </collision>
             <xacro:wheel_inertia  m="1.0" r="${wheel_radius}" l="${wheel_length}"
                                     xyz="0 0 0" rpy="${pi/2.0} 0 0"/>
@@ -57,5 +69,11 @@
             <material name="grey"/>
         </visual>
-        <xacro:wheel_inertia  m="0.5" r="${wheel_radius/2}" xyz="0 0 0" rpy="0 0 0"/>
+        <collision>
+            <geometry>
+                <sphere radius="${wheel_radius/2}"/>
+            </geometry>
+            <origin xyz="0 0 0" rpy="0 0 0"/>
+        </collision>
+        <xacro:caster_wheel_inertia  m="0.5" r="${wheel_radius/2}" xyz="0 0 0" rpy="0 0 0"/>
     </link>
     <joint name = "base_joint" type="fixed">

Commit message: ros_gazebo_bridge established!

File: src/my_robot_description/urdf/mobile_base.xacro (robot description, xacro)
@@ -6,4 +6,10 @@
     <xacro:property name="wheel_radius" value="0.1"/>
     <xacro:property name="wheel_length" value="0.05"/>
+    <link name="base_footprint" />
+    <joint name = "base_joint" type="fixed">
+        <parent link="base_footprint"/>
+        <child link = "base_link"/>
+        <origin xyz="0 0 ${wheel_radius}" rpy="0 0 0"/>
+    </joint>
     <link name="base_link">
         <visual>
@@ -77,9 +83,3 @@
         <xacro:caster_wheel_inertia  m="0.5" r="${wheel_radius/2}" xyz="0 0 0" rpy="0 0 0"/>
     </link>
-    <joint name = "base_joint" type="fixed">
-        <parent link="world"/>
-        <child link = "base_link"/>
-        <origin xyz="0 0 ${wheel_radius}" rpy="0 0 0"/>
-    </joint>
-    <link name="world" />
 </robot>

File: src/my_robot_description/urdf/my_robot.urdf.xacro (robot description, xacro)
@@ -3,3 +3,4 @@
 <xacro:include filename="$(find my_robot_description)/urdf/common_properties.xacro"/>
 <xacro:include filename="$(find my_robot_description)/urdf/mobile_base.xacro"/>
+<xacro:include filename="$(find my_robot_description)/urdf/mobile_base_gazebo.xacro"/>
 </robot>
