Commit message: camera sensor update

File: src/my_robot_description/urdf/camera.xacro (robot description, xacro)
@@ -4,4 +4,10 @@
     <xacro:property name="camera_width" value="0.1" />
     <xacro:property name="camera_height" value="0.05" />
+    <link name="camera_link_optical"/>
+    <joint name="camera_optical_joint" type="fixed">
+      <origin xyz="0 0 0" rpy="${-pi/2} 0 ${-pi/2}"/>
+      <parent link="camera_link"/>
+      <child link="camera_link_optical"/>
+    </joint>
     <link name="camera_link">
         <visual>
@@ -26,18 +32,26 @@
         <sensor name="camera_sensor" type="camera">
           <camera>
-            <horizontal_fov>1.047</horizontal_fov>
+            <horizontal_fov>1.3962634</horizontal_fov>
             <image>
-              <width>320</width>
-              <height>240</height>
+              <width>640</width>
+              <height>480</height>
+              <format>R8G8B8</format>
             </image>
             <clip>
               <near>0.1</near>
-              <far>100</far>
+              <far>15</far>
             </clip>
+            <noise>
+              <type>gaussian</type>
+              <mean>0.0</mean>
+              <stddev>0.007</stddev>
+            </noise>
+            <optical_frame_id>camera_link_optical</optical_frame_id>
+            <camera_info_topic>camera/camera_info</camera_info_topic>
           </camera>
           <always_on>1</always_on>
           <update_rate>30</update_rate>
           <visualize>true</visualize>
-          <topic>camera</topic>
+          <topic>camera/image_raw </topic>
         </sensor>
     </gazebo>
