Commit message: inertial properties added to the link

File: src/my_robot_description/urdf/common_properties.xacro (robot description, xacro)
@@ -7,3 +7,30 @@
         <color rgba="0.5 0.5 0.5 1"/>
     </material>
+    <xacro:macro name="box_inertia" params="m l w h xyz rpy">
+        <inertia>
+            <mass value="${m}" />
+            <origin xyz="${xyz}" rpy ="${rpy}" />
+            <inertia ixx="${(m/12) * (h*h + l*l)}" ixy="0" ixz="0"
+                     iyy="${(m/12) * (w*w + l*l)}" iyz ="0"
+                     izz="${(m/12) * (h*h + w*w )}" />
+        </inertia>
+    </xacro:macro>
+    <xacro:macro name="wheel_inertia" params="m r l xyz rpy">
+        <inertia>
+            <mass value="${m}" />
+            <origin xyz="${xyz}" rpy ="${rpy}" />
+            <inertia ixx="${(m/12) * (3*r*r + l*l)}" ixy="0" ixz="0"
+                     iyy="${(m/12) * (3*r*r + l*l)}" iyz ="0"
+                     izz="${m*r*r/2}" />
+        </inertia>
+    </xacro:macro>
+    <xacro:macro name="caster_wheel_inertia" params="m r xyz rpy">
+        <inertia>
+            <mass value="${m}" />
+            <origin xyz="${xyz}" rpy ="${rpy}" />
+            <inertia ixx="${2/5*m*r*r}" ixy="0" ixz="0"
+                     iyy="${2/5*m*r*r}" iyz ="0"
+                     izz="${2/5*m*r*r}" />
+        </inertia>
+    </xacro:macro>
 </robot>

File: src/my_robot_description/urdf/mobile_base.xacro (robot description, xacro)
@@ -14,4 +14,6 @@
             <material name="blue" />
         </visual>
+        <xacro:box_inertia  m="5" l="${base_length}" w="${base_width}" h="${base_height}"
+                            xyz="0 0 ${base_height/2.0}" rpy="0 0 0"/>
     </link>
     <joint name = "base_right_wheel_joint" type="continuous">
@@ -30,4 +32,6 @@
                 <material name="grey"/>
             </visual>
+            <xacro:wheel_inertia  m="1.0" r="${wheel_radius}" l="${wheel_length}"
+                                    xyz="0 0 0" rpy="${pi/2.0} 0 0"/>
         </link>
     </xacro:macro>
@@ -53,4 +57,5 @@
             <material name="grey"/>
         </visual>
+        <xacro:wheel_inertia  m="0.5" r="${wheel_radius/2}" xyz="0 0 0" rpy="0 0 0"/>
     </link>
     <joint name = "base_joint" type="fixed">

Commit message: integration of two independent robotic systems - ROS2 + Gazebo sim Final Project (Humble, Fortress)

File: src/my_robot_description/urdf/common_properties.xacro (robot description, xacro)
@@ -6,4 +6,10 @@
     <material name="grey">
         <color rgba="0.5 0.5 0.5 1"/>
+    </material>
+    <material name="orange">
+        <color rgba="1.0 0.5 0 1"/>
+    </material>
+    <material name="yellow">
+        <color rgba="1.0 1.0 0 1"/>
     </material>
     <xacro:macro name="box_inertia" params="m l w h xyz rpy">

File: src/my_robot_description/urdf/mobile_base.xacro (robot description, xacro)
@@ -26,5 +26,5 @@
             <origin xyz="0 0 ${base_height / 2.0}" rpy="0 0 0" />
         </collision>
-        <xacro:box_inertia  m="5" l="${base_length}" w="${base_width}" h="${base_height}"
+        <xacro:box_inertia  m="0.5" l="${base_length}" w="${base_width}" h="${base_height}"
                             xyz="0 0 ${base_height/2.0}" rpy="0 0 0"/>
     </link>

File: src/my_robot_description/urdf/mobile_base_gazebo.xacro (robot description, xacro)
@@ -29,5 +29,5 @@
           <render_engine>ogre2</render_engine>
         <frame_id>odom</frame_id>
-          <child_frame_id>base_link</child_frame_id>
+        <child_frame_id>base_link</child_frame_id>
         </plugin>
     </gazebo>

File: src/my_robot_description/urdf/my_robot.urdf.xacro (robot description, xacro)
@@ -3,5 +3,12 @@
 <xacro:include filename="$(find my_robot_description)/urdf/common_properties.xacro"/>
 <xacro:include filename="$(find my_robot_description)/urdf/mobile_base.xacro"/>
+<xacro:include filename="$(find my_robot_description)/urdf/camera.xacro"/>
 <xacro:include filename="$(find my_robot_description)/urdf/mobile_base_gazebo.xacro"/>
-<xacro:include filename="$(find my_robot_description)/urdf/camera.xacro"/>
+<xacro:include filename="$(find my_robot_description)/urdf/mobile_arm.xacro"/>
+<xacro:include filename="$(find my_robot_description)/urdf/arm_gazebo.xacro"/>
+<joint name = "arm_base_joint" type="fixed">
+    <parent link="base_link"/>
+    <child link = "arm_base_footprint"/>
+    <origin xyz="${base_length/2 - arm_base_length/2} 0 ${base_height+arm_base_height/2}" rpy="0 0 0"/>
+</joint>
 </robot>
