Commit message: finally inside gazebo fortress!

File: install/my_robot_description/share/my_robot_description/urdf/common_properties.xacro (robot description, xacro)
@@ -1,36 +1 @@
-<?xml version="1.0"?>
-<robot xmlns:xacro="https://www.ros.org/wiki/xacro">
-    <material name="blue">
-        <color rgba="0 0 0.5 1"/>
-    </material>
-    <material name="grey">
-        <color rgba="0.5 0.5 0.5 1"/>
-    </material>
-    <xacro:macro name="box_inertia" params="m l w h xyz rpy">
-        <inertia>
-            <mass value="${m}" />
-            <origin xyz="${xyz}" rpy ="${rpy}" />
-            <inertia ixx="${(m/12) * (h*h + l*l)}" ixy="0" ixz="0"
-                     iyy="${(m/12) * (w*w + l*l)}" iyz ="0"
-                     izz="${(m/12) * (h*h + w*w )}" />
-        </inertia>
-    </xacro:macro>
-    <xacro:macro name="wheel_inertia" params="m r l xyz rpy">
-        <inertia>
-            <mass value="${m}" />
-            <origin xyz="${xyz}" rpy ="${rpy}" />
-            <inertia ixx="${(m/12) * (3*r*r + l*l)}" ixy="0" ixz="0"
-                     iyy="${(m/12) * (3*r*r + l*l)}" iyz ="0"
-                     izz="${m*r*r/2}" />
-        </inertia>
-    </xacro:macro>
-    <xacro:macro name="caster_wheel_inertia" params="m r xyz rpy">
-        <inertia>
-            <mass value="${m}" />
-            <origin xyz="${xyz}" rpy ="${rpy}" />
-            <inertia ixx="${2/5*m*r*r}" ixy="0" ixz="0"
-                     iyy="${2/5*m*r*r}" iyz ="0"
-                     izz="${2/5*m*r*r}" />
-        </inertia>
-    </xacro:macro>
-</robot>
+/home/parallels/ros2_ws/src/my_robot_description/urdf/common_properties.xacro

File: install/my_robot_description/share/my_robot_description/urdf/mobile_base.xacro (robot description, xacro)
@@ -1,89 +1 @@
-<?xml version="1.0"?>
-<robot xmlns:xacro="https://www.ros.org/wiki/xacro">
-    <xacro:property name="base_length" value="0.6"/>
-    <xacro:property name="base_width" value="0.4"/>
-    <xacro:property name="base_height" value="0.2"/>
-    <xacro:property name="wheel_radius" value="0.1"/>
-    <xacro:property name="wheel_length" value="0.05"/>
-    <link name="base_link">
-        <visual>
-            <geometry>
-                <box size="${base_length} ${base_width} ${base_height}" />
-            </geometry>
-            <origin xyz="0 0 ${base_height/2.0}" rpy="0 0 0" />
-            <material name="blue" />
-        </visual>
-        <collision>
-            <geometry>
-                <box size="${base_length} ${base_width} ${base_height}" />
-            </geometry>
-            <origin xyz="0 0 ${base_height / 2.0}" rpy="0 0 0" />
-        </collision>
-        <xacro:box_inertia  m="5" l="${base_length}" w="${base_width}" h="${base_height}"
-                            xyz="0 0 ${base_height/2.0}" rpy="0 0 0"/>
-    </link>
-    <joint name = "base_right_wheel_joint" type="continuous">
-        <parent link="base_link"/>
-        <child link = "right_wheel_link"/>
-        <origin xyz="${-base_length/4} ${-base_width/1.7778} 0" rpy="0 0 0"/>
-        <axis xyz="0 1 0"/>
-    </joint>
-    <xacro:macro name="wheel_link" params="prefix">
-        <link name="${prefix}_wheel_link">
-            <visual>
-                <geometry>
-                    <cylinder radius="${wheel_radius}" length="${wheel_length}"/>
-                </geometry>
-                <origin xyz="0 0 0" rpy="${pi/2.0} 0 0"/>
-                <material name="grey"/>
-            </visual>
-            <collision>
-                <geometry>
-                    <cylinder radius="${wheel_radius}" length="${wheel_length}"/>
-                </geometry>
-                <origin xyz="0 0 0" rpy="${pi/2.0} 0 0"/>
-            </collision>
-            <xacro:wheel_inertia  m="1.0" r="${wheel_radius}" l="${wheel_length}"
-                                    xyz="0 0 0" rpy="${pi/2.0} 0 0"/>
-        </link>
-    </xacro:macro>
-    <xacro:wheel_link prefix="right"/>
-    <joint name = "base_left_wheel_joint" type="continuous">
-        <parent link="base_link"/>
-        <child link = "left_wheel_link"/>
-        <origin xyz="${-base_length/4} ${base_width/1.7778} 0" rpy="0 0 0"/>
-        <axis xyz="0 1 0"/>
-    </joint>
-    <xacro:wheel_link prefix="left"/>
-    <joint name = "base_caster_wheel_joint" type="fixed">
-        <parent link="base_link"/>
-        <child link = "caster_wheel_link"/>
-        <origin xyz="${base_length/3} 0 ${-wheel_radius/2} " rpy="0 0 0"/>
-    </joint>
-    <link name="caster_wheel_link">
-        <visual>
-            <geometry>
-                <sphere radius="${wheel_radius/2}"/>
-            </geometry>
-            <origin xyz="0 0 0" rpy="0 0 0"/>
-            <material name="grey"/>
-        </visual>
-        <collision>
-            <geometry>
-                <sphere radius="${wheel_radius/2}"/>
-            </geometry>
-            <origin xyz="0 0 0" rpy="0 0 0"/>
-        </collision>
-        <xacro:caster_wheel_inertia  m="0.5" r="${wheel_radius/2}" xyz="0 0 0" rpy="0 0 0"/>
-    </link>
-    <joint name = "base_joint" type="fixed">
-        <parent link="base_footprint"/>
-        <child link = "base_link"/>
-        <origin xyz="0 0 ${wheel_radius}" rpy="0 0 0"/>
-    </joint>
-    <link name="base_footprint">
-        <visual>
-            <origin xyz="0 0 0" rpy="0 0 0"/>
-        </visual>
-    </link>
-</robot>
+/home/parallels/ros2_ws/src/my_robot_description/urdf/mobile_base.xacro

File: install/my_robot_description/share/my_robot_description/urdf/my_robot.urdf.xacro (robot description, xacro)
@@ -1,5 +1 @@
-<?xml version="1.0"?>
-<robot name="my_robot" xmlns:xacro="https://www.ros.org/wiki/xacro">
-    <xacro:include filename="common_properties.xacro"/>
-    <xacro:include filename="mobile_base.xacro"/>
-</robot>
+/home/parallels/ros2_ws/src/my_robot_description/urdf/my_robot.urdf.xacro

File: src/my_robot_description/urdf/common_properties.xacro (robot description, xacro)
@@ -1,4 +1,4 @@
 <?xml version="1.0"?>
-<robot xmlns:xacro="https://www.ros.org/wiki/xacro">
+<robot xmlns:xacro="http://www.ros.org/wiki/xacro">
     <material name="blue">
         <color rgba="0 0 0.5 1"/>
@@ -8,5 +8,5 @@
     </material>
     <xacro:macro name="box_inertia" params="m l w h xyz rpy">
-        <inertia>
+        <inertial>
             <mass value="${m}" />
             <origin xyz="${xyz}" rpy ="${rpy}" />
@@ -14,8 +14,8 @@
                      iyy="${(m/12) * (w*w + l*l)}" iyz ="0"
                      izz="${(m/12) * (h*h + w*w )}" />
-        </inertia>
+        </inertial>
     </xacro:macro>
     <xacro:macro name="wheel_inertia" params="m r l xyz rpy">
-        <inertia>
+        <inertial>
             <mass value="${m}" />
             <origin xyz="${xyz}" rpy ="${rpy}" />
@@ -23,8 +23,8 @@
                      iyy="${(m/12) * (3*r*r + l*l)}" iyz ="0"
                      izz="${m*r*r/2}" />
-        </inertia>
+        </inertial>
     </xacro:macro>
     <xacro:macro name="caster_wheel_inertia" params="m r xyz rpy">
-        <inertia>
+        <inertial>
             <mass value="${m}" />
             <origin xyz="${xyz}" rpy ="${rpy}" />
@@ -32,5 +32,5 @@
                      iyy="${2/5*m*r*r}" iyz ="0"
                      izz="${2/5*m*r*r}" />
-        </inertia>
+        </inertial>
     </xacro:macro>
 </robot>

File: src/my_robot_description/urdf/mobile_base.xacro (robot description, xacro)
@@ -1,4 +1,4 @@
 <?xml version="1.0"?>
-<robot xmlns:xacro="https://www.ros.org/wiki/xacro">
+<robot xmlns:xacro="http://www.ros.org/wiki/xacro">
     <xacro:property name="base_length" value="0.6"/>
     <xacro:property name="base_width" value="0.4"/>
@@ -78,12 +78,8 @@
     </link>
     <joint name = "base_joint" type="fixed">
-        <parent link="base_footprint"/>
+        <parent link="world"/>
         <child link = "base_link"/>
         <origin xyz="0 0 ${wheel_radius}" rpy="0 0 0"/>
     </joint>
-    <link name="base_footprint">
-        <visual>
-            <origin xyz="0 0 0" rpy="0 0 0"/>
-        </visual>
-    </link>
+    <link name="world" />
 </robot>

File: src/my_robot_description/urdf/my_robot.urdf.xacro (robot description, xacro)
@@ -1,5 +1,5 @@
 <?xml version="1.0"?>
-<robot name="my_robot" xmlns:xacro="https://www.ros.org/wiki/xacro">
-    <xacro:include filename="common_properties.xacro"/>
-    <xacro:include filename="mobile_base.xacro"/>
+<robot name="my_robot" xmlns:xacro="http://www.ros.org/wiki/xacro">
+<xacro:include filename="$(find my_robot_description)/urdf/common_properties.xacro"/>
+<xacro:include filename="$(find my_robot_description)/urdf/mobile_base.xacro"/>
 </robot>
