Commit message: lifecycle_node_launch

File: install/my_robot_description/share/my_robot_description/urdf/arm_gazebo.xacro (robot description, xacro)
@@ -1 +1,23 @@
-/home/parallels/ros2_ws/src/my_robot_description/urdf/arm_gazebo.xacro
+<?xml version="1.0"?>
+<robot xmlns:xacro="http://www.ros.org/wiki/xacro">
+    <gazebo>
+        <plugin
+            filename="gz-sim-joint-position-controller-system"
+            name="gz::sim::systems::JointPositionController">
+            <joint_name>base_forarm_joint</joint_name>
+        </plugin>
+        <plugin
+            filename="gz-sim-joint-position-controller-system"
+            name="gz::sim::systems::JointPositionController">
+            <joint_name>forearm_hand_joint</joint_name>
+        </plugin>
+    </gazebo>
+    <gazebo>
+        <plugin
+            filename="gz-sim-joint-state-publisher-system"
+            name="gz::sim::systems::JointStatePublisher">
+            <joint_name>base_forarm_joint</joint_name>
+            <joint_name>forearm_hand_joint</joint_name>
+        </plugin>
+    </gazebo>
+</robot>

File: install/my_robot_description/share/my_robot_description/urdf/camera.xacro (robot description, xacro)
@@ -1 +1,58 @@
-/home/parallels/ros2_ws/src/my_robot_description/urdf/camera.xacro
+<?xml version="1.0"?>
+<robot name="my_robot" xmlns:xacro="http://www.ros.org/wiki/xacro">
+    <xacro:property name="camera_length" value="0.01" />
+    <xacro:property name="camera_width" value="0.1" />
+    <xacro:property name="camera_height" value="0.05" />
+    <link name="camera_link_optical"/>
+    <joint name="camera_optical_joint" type="fixed">
+      <origin xyz="0 0 0" rpy="${-pi/2} 0 ${-pi/2}"/>
+      <parent link="camera_link"/>
+      <child link="camera_link_optical"/>
+    </joint>
+    <link name="camera_link">
+        <visual>
+            <geometry>
+                <box size ="${camera_length} ${camera_width} ${camera_height}"/>
+            </geometry>
+            <material name="grey"/>
+        </visual>
+        <collision>
+            <geometry>
+                <box size ="${camera_length} ${camera_width} ${camera_height}"/>
+            </geometry>
+        </collision>
+        <xacro:box_inertia m = "0.1" l="${camera_length}" w="${camera_width}" h="${camera_height}" xyz="0 0 0" rpy="0 0 0"/>
+    </link>
+    <joint name="base_camera_joint" type="fixed">
+        <parent link="base_link"/>
+        <child link="camera_link"/>
+        <origin xyz="${base_length/2+camera_length} 0 ${base_height/2}" rpy="0 0 0"/>
+    </joint>
+    <gazebo reference="camera_link">
+        <sensor name="camera_sensor" type="camera">
+          <camera>
+            <horizontal_fov>1.3962634</horizontal_fov>
+            <image>
+              <width>640</width>
+              <height>480</height>
+              <format>R8G8B8</format>
+            </image>
+            <clip>
+              <near>0.1</near>
+              <far>15</far>
+            </clip>
+            <noise>
+              <type>gaussian</type>
+              <mean>0.0</mean>
+              <stddev>0.007</stddev>
+            </noise>
+            <optical_frame_id>camera_link_optical</optical_frame_id>
+            <camera_info_topic>camera/camera_info</camera_info_topic>
+          </camera>
+          <always_on>1</always_on>
+          <update_rate>30</update_rate>
+          <visualize>true</visualize>
+          <topic>camera/image_raw </topic>
+        </sensor>
+    </gazebo>
+</robot>

File: install/my_robot_description/share/my_robot_description/urdf/common_properties.xacro (robot description, xacro)
@@ -1 +1,42 @@
-/home/parallels/ros2_ws/src/my_robot_description/urdf/common_properties.xacro
+<?xml version="1.0"?>
+<robot xmlns:xacro="http://www.ros.org/wiki/xacro">
+    <material name="blue">
+        <color rgba="0 0 0.5 1"/>
+    </material>
+    <material name="grey">
+        <color rgba="0.5 0.5 0.5 1"/>
+    </material>
+    <material name="orange">
+        <color rgba="1.0 0.5 0 1"/>
+    </material>
+    <material name="yellow">
+        <color rgba="1.0 1.0 0 1"/>
+    </material>
+    <xacro:macro name="box_inertia" params="m l w h xyz rpy">
+        <inertial>
+            <mass value="${m}" />
+            <origin xyz="${xyz}" rpy ="${rpy}" />
+            <inertia ixx="${(m/12) * (h*h + l*l)}" ixy="0" ixz="0"
+                     iyy="${(m/12) * (w*w + l*l)}" iyz ="0"
+                     izz="${(m/12) * (h*h + w*w )}" />
+        </inertial>
+    </xacro:macro>
+    <xacro:macro name="wheel_inertia" params="m r l xyz rpy">
+        <inertial>
+            <mass value="${m}" />
+            <origin xyz="${xyz}" rpy ="${rpy}" />
+            <inertia ixx="${(m/12) * (3*r*r + l*l)}" ixy="0" ixz="0"
+                     iyy="${(m/12) * (3*r*r + l*l)}" iyz ="0"
+                     izz="${m*r*r/2}" />
+        </inertial>
+    </xacro:macro>
+    <xacro:macro name="caster_wheel_inertia" params="m r xyz rpy">
+        <inertial>
+            <mass value="${m}" />
+            <origin xyz="${xyz}" rpy ="${rpy}" />
+            <inertia ixx="${2/5*m*r*r}" ixy="0" ixz="0"
+                     iyy="${2/5*m*r*r}" iyz ="0"
+                     izz="${2/5*m*r*r}" />
+        </inertial>
+    </xacro:macro>
+</robot>

File: install/my_robot_description/share/my_robot_description/urdf/mobile_arm.urdf.xacro (robot description, xacro)
@@ -1 +1,6 @@
-/home/parallels/ros2_ws/src/my_robot_description/urdf/mobile_arm.urdf.xacro
+<?xml version="1.0"?>
+<robot name="my_robot" xmlns:xacro="http://www.ros.org/wiki/xacro">
+<xacro:include filename="$(find my_robot_description)/urdf/common_properties.xacro"/>
+<xacro:include filename="$(find my_robot_description)/urdf/mobile_arm.xacro"/>
+<xacro:include filename="$(find my_robot_description)/urdf/arm_gazebo.xacro"/>
+</robot>

File: install/my_robot_description/share/my_robot_description/urdf/mobile_arm.xacro (robot description, xacro)
@@ -1 +1,83 @@
-/home/parallels/ros2_ws/src/my_robot_description/urdf/mobile_arm.xacro
+<?xml version="1.0"?>
+<robot name="my_robot" xmlns:xacro="http://www.ros.org/wiki/xacro">
+    <xacro:property name="arm_base_length" value="0.1"/>
+    <xacro:property name="arm_base_width" value="0.1"/>
+    <xacro:property name="arm_base_height" value="0.02"/>
+    <xacro:property name="forearm_link_radius" value="0.02"/>
+    <xacro:property name="forearm_link_length" value="0.3"/>
+    <xacro:property name="hand_link_radius" value="0.02"/>
+    <xacro:property name="hand_link_length" value="0.3"/>
+        <link name="arm_base_footprint"/>
+        <joint name = "base_footprint_arm_joint" type="fixed">
+            <parent link="arm_base_footprint"/>
+            <child link = "arm_base_link"/>
+            <origin xyz="0 0 0" rpy="0 0 0"/>
+        </joint>
+        <link name="arm_base_link">
+            <visual>
+                <geometry>
+                    <box size="${arm_base_length} ${arm_base_width} ${arm_base_height}" />
+                </geometry>
+                <origin xyz="0 0 0" rpy="0 0 0" />
+                <material name="orange"/>
+            </visual>
+            <collision>
+                <geometry>
+                    <box size="${arm_base_length} ${arm_base_width} ${arm_base_height}" />
+                </geometry>
+                <origin xyz="0 0 0" rpy="0 0 0" />
+            </collision>
+            <xacro:box_inertia  m="0.5" l="${arm_base_length}" w="${arm_base_width}" h="${arm_base_height}"
+                                xyz="0 0 0" rpy="${pi/2} 0 0"/>
+        </link>
+        <joint name = "base_forarm_joint" type="revolute">
+            <parent link="arm_base_link"/>
+            <child link = "forearm_link"/>
+            <origin xyz="0 0 ${arm_base_height/2}" rpy="0 0 0"/>
+            <axis xyz="0 1 0"/>
+            <dynamics damping="0.1" friction="0.1"/>
+            <limit lower="0" upper="${pi/2}" effort="100" velocity="100"/>
+        </joint>
+        <link name="forearm_link">
+            <visual>
+                <geometry>
+                    <cylinder radius="${forearm_link_radius}" length="${forearm_link_length}" />
+                </geometry>
+                <origin xyz="0 0 ${forearm_link_length/2.0}" rpy="0 0 0" />
+                <material name="yellow"/>
+            </visual>
+            <collision>
+                <geometry>
+                    <cylinder radius="${forearm_link_radius}" length="${forearm_link_length}" />
+                </geometry>
+                <origin xyz="0 0 ${forearm_link_length/2.0}" rpy="0 0 0" />
+            </collision>
+            <xacro:wheel_inertia  m="0.3" r="${forearm_link_radius}" l="${forearm_link_length}"
+                                    xyz="0 0 ${forearm_link_length/2.0}" rpy="0 0 0"/>
+        </link>
+        <link name="hand_link">
+            <visual>
+                <geometry>
+                    <cylinder radius="${hand_link_radius}" length="${hand_link_length}" />
+                </geometry>
+                <origin xyz="0 0 ${hand_link_length/2.0}" rpy="0 0 0" />
+                <material name="orange"/>
+            </visual>
+            <collision>
+                <geometry>
+                    <cylinder radius="${hand_link_radius}" length="${hand_link_length}" />
+                </geometry>
+                <origin xyz="0 0 ${hand_link_length/2.0}" rpy="0 0 0" />
+            </collision>
+            <xacro:wheel_inertia  m="0.3" r="${hand_link_radius}" l="${hand_link_length}"
+                                    xyz="0 0 ${hand_link_length/2.0}" rpy="0 0 0"/>
+        </link>
+        <joint name = "forearm_hand_joint" type="revolute">
+            <parent link="forearm_link"/>
+            <child link = "hand_link"/>
+            <origin xyz="0 0 ${hand_link_length}" rpy="0 0 0"/>
+            <axis xyz="0 1 0"/>
+            <dynamics damping="0.1" friction="0.1"/>
+            <limit lower="0" upper="${pi/2}" effort="100" velocity="100"/>
+        </joint>
+</robot>

File: install/my_robot_description/share/my_robot_description/urdf/mobile_base.xacro (robot description, xacro)
@@ -1 +1,85 @@
-/home/parallels/ros2_ws/src/my_robot_description/urdf/mobile_base.xacro
+<?xml version="1.0"?>
+<robot xmlns:xacro="http://www.ros.org/wiki/xacro">
+    <xacro:property name="base_length" value="0.6"/>
+    <xacro:property name="base_width" value="0.4"/>
+    <xacro:property name="base_height" value="0.2"/>
+    <xacro:property name="wheel_radius" value="0.1"/>
+    <xacro:property name="wheel_length" value="0.05"/>
+    <link name="base_footprint" />
+    <joint name = "base_joint" type="fixed">
+        <parent link="base_footprint"/>
+        <child link = "base_link"/>
+        <origin xyz="0 0 ${wheel_radius}" rpy="0 0 0"/>
+    </joint>
+    <link name="base_link">
+        <visual>
+            <geometry>
+                <box size="${base_length} ${base_width} ${base_height}" />
+            </geometry>
+            <origin xyz="0 0 ${base_height/2.0}" rpy="0 0 0" />
+            <material name="blue" />
+        </visual>
+        <collision>
+            <geometry>
+                <box size="${base_length} ${base_width} ${base_height}" />
+            </geometry>
+            <origin xyz="0 0 ${base_height / 2.0}" rpy="0 0 0" />
+        </collision>
+        <xacro:box_inertia  m="0.5" l="${base_length}" w="${base_width}" h="${base_height}"
+                            xyz="0 0 ${base_height/2.0}" rpy="0 0 0"/>
+    </link>
+    <xacro:macro name="wheel_link" params="prefix">
+        <link name="${prefix}_wheel_link">
+            <visual>
+                <geometry>
+                    <cylinder radius="${wheel_radius}" length="${wheel_length}"/>
+                </geometry>
+                <origin xyz="0 0 0" rpy="${pi/2.0} 0 0"/>
+                <material name="grey"/>
+            </visual>
+            <collision>
+                <geometry>
+                    <cylinder radius="${wheel_radius}" length="${wheel_length}"/>
+                </geometry>
+                <origin xyz="0 0 0" rpy="${pi/2.0} 0 0"/>
+            </collision>
+            <xacro:wheel_inertia  m="1.0" r="${wheel_radius}" l="${wheel_length}"
+                                    xyz="0 0 0" rpy="${pi/2.0} 0 0"/>
+        </link>
+    </xacro:macro>
+    <joint name = "base_right_wheel_joint" type="continuous">
+        <parent link="base_link"/>
+        <child link = "right_wheel_link"/>
+        <origin xyz="${-base_length/4} ${-base_width/1.7778} 0" rpy="0 0 0"/>
+        <axis xyz="0 1 0"/>
+    </joint>
+    <xacro:wheel_link prefix="right"/>
+    <joint name = "base_left_wheel_joint" type="continuous">
+        <parent link="base_link"/>
+        <child link = "left_wheel_link"/>
+        <origin xyz="${-base_length/4} ${base_width/1.7778} 0" rpy="0 0 0"/>
+        <axis xyz="0 1 0"/>
+    </joint>
+    <xacro:wheel_link prefix="left"/>
+    <joint name = "base_caster_wheel_joint" type="fixed">
+        <parent link="base_link"/>
+        <child link = "caster_wheel_link"/>
+        <origin xyz="${base_length/3} 0 ${-wheel_radius/2} " rpy="0 0 0"/>
+    </joint>
+    <link name="caster_wheel_link">
+        <visual>
+            <geometry>
+                <sphere radius="${wheel_radius/2}"/>
+            </geometry>
+            <origin xyz="0 0 0" rpy="0 0 0"/>
+            <material name="grey"/>
+        </visual>
+        <collision>
+            <geometry>
+                <sphere radius="${wheel_radius/2}"/>
+            </geometry>
+            <origin xyz="0 0 0" rpy="0 0 0"/>
+        </collision>
+        <xacro:caster_wheel_inertia  m="0.5" r="${wheel_radius/2}" xyz="0 0 0" rpy="0 0 0"/>
+    </link>
+</robot>

File: install/my_robot_description/share/my_robot_description/urdf/mobile_base_gazebo.xacro (robot description, xacro)
@@ -1 +1,34 @@
-/home/parallels/ros2_ws/src/my_robot_description/urdf/mobile_base_gazebo.xacro
+<?xml version="1.0"?>
+<robot xmlns:xacro="http://www.ros.org/wiki/xacro">
+    <gazebo reference='base_link'>
+        <material>Gazebo/Orange</material>
+    </gazebo>
+    <gazebo reference="caster_wheel_link">
+        <mu1 value="0.1" />
+        <mu2 value="0.1" />
+    </gazebo>
+    <gazebo>
+        <plugin
+            filename="gz-sim-diff-drive-system"
+            name="gz::sim::systems::DiffDrive">
+            <update_rate>50</update_rate>
+            <left_joint>base_left_wheel_joint</left_joint>
+            <right_joint>base_right_wheel_joint</right_joint>
+            <frame_id>odom</frame_id>
+            <child_frame_id>base_footprint</child_frame_id>
+            <wheel_separation>0.45</wheel_separation>
+            <wheel_radius>0.1</wheel_radius>
+        </plugin>
+        <plugin
+            filename="gz-sim-joint-state-publisher-system"
+            name="gz::sim::systems::JointStatePublisher">
+        </plugin>
+        <plugin
+          filename="gz-sim-sensors-system"
+          name="gz::sim::systems::Sensors">
+          <render_engine>ogre2</render_engine>
+        <frame_id>odom</frame_id>
+        <child_frame_id>base_link</child_frame_id>
+        </plugin>
+    </gazebo>
+</robot>

File: install/my_robot_description/share/my_robot_description/urdf/my_robot.urdf.xacro (robot description, xacro)
@@ -1 +1,14 @@
-/home/parallels/ros2_ws/src/my_robot_description/urdf/my_robot.urdf.xacro
+<?xml version="1.0"?>
+<robot name="my_robot" xmlns:xacro="http://www.ros.org/wiki/xacro">
+<xacro:include filename="$(find my_robot_description)/urdf/common_properties.xacro"/>
+<xacro:include filename="$(find my_robot_description)/urdf/mobile_base.xacro"/>
+<xacro:include filename="$(find my_robot_description)/urdf/camera.xacro"/>
+<xacro:include filename="$(find my_robot_description)/urdf/mobile_base_gazebo.xacro"/>
+<xacro:include filename="$(find my_robot_description)/urdf/mobile_arm.xacro"/>
+<xacro:include filename="$(find my_robot_description)/urdf/arm_gazebo.xacro"/>
+<joint name = "arm_base_joint" type="fixed">
+    <parent link="base_link"/>
+    <child link = "arm_base_footprint"/>
+    <origin xyz="${base_length/2 - arm_base_length/2} 0 ${base_height+arm_base_height/2}" rpy="0 0 0"/>
+</joint>
+</robot>
