Commit message: FIx: Moveit2 tutorials patched for the moveit2 kilted

File: my_robot_description/urdf/my_robot_base_arm.urdf.xacro (robot description, xacro)
@@ -4,12 +4,12 @@
 <xacro:include filename="$(find my_robot_description)/urdf/mobile_base.xacro"/>
 <xacro:include filename="$(find my_robot_description)/urdf/camera.xacro"/>
-<xacro:include filename="$(find my_robot_description)/urdf/mobile_arm.xacro"/>
+<!-- <xacro:include filename="$(find my_robot_description)/urdf/mobile_arm.xacro"/> -->
 <xacro:include filename="$(find my_robot_description)/urdf/mobile_base_gazebo.xacro"/>
 <!-- <xacro:include filename="$(find my_robot_description)/urdf/arm_gazebo.xacro"/> -->
 <!-- <xacro:include filename="$(find my_robot_description)/urdf/my_controllers.urdf.xacro"/> -->
-<joint name = "arm_base_joint" type="fixed">
+<!-- <joint name = "arm_base_joint" type="fixed">
     <parent link="base_link"/>
     <child link = "arm_base_footprint"/>
     <origin xyz="${base_length/2 - arm_base_length/2} 0 ${base_height+arm_base_height/2}" rpy="0 0 0"/>
-</joint>
+</joint> -->
 </robot>
